Commit message: removing imu_link from urdf

File: husky_description/urdf/husky.urdf.xacro (robot description, xacro)
@@ -91,5 +91,5 @@
   <!-- IMU Link is the standard mounting position for the UM6 IMU.-->
   <!-- Can be modified with environment variables in /etc/ros/setup.bash -->
-  <link name="imu_link"/>
+<!--   <link name="imu_link"/>
   <joint name="imu_joint" type="fixed">
     <origin xyz="$(optenv HUSKY_IMU_XYZ 0.19 0 0.149)" rpy="$(optenv HUSKY_IMU_RPY 0 -1.5708 3.1416)" />
@@ -98,5 +98,5 @@
   </joint>
   <gazebo reference="imu_link">
-  </gazebo>
+  </gazebo> -->
   <!-- Husky wheel macros -->
   <xacro:husky_wheel wheel_prefix="front_left">
